File: bitaxeGamma.kicad_sch (KiCad schematic)
At the start: 20 parts, among them J1 54-00164

Commit message: switching to gamma/600 naming
Other:
- sheet BM1368 renamed BM1370
- sheet BM1370: file bm1368.kicad_sch -> bm1370.kicad_sch
- title: bitaxeSupra -> bitaxeGamma
Changed lines of the file:
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@@
 	(paper "A")
 	(title_block
-		(title "bitaxeSupra")
-		(date "2024-04-07")
-		(rev "402")
+		(title "bitaxeGamma")
+		(date "2024-07-02")
+		(rev "600x")
 	)
 	(junction
@@
 		)
 		(instances
-			(project "bitaxeSupra"
+			(project "bitaxeGamma"
 				(path "/e63e39d7-6ac0-4ffd-8aa3-1841a4541b55"
 					(reference "FID2")
@@
 		)
 		(instances
-			(project "bitaxeSupra"
+			(project "bitaxeGamma"
 				(path "/e63e39d7-6ac0-4ffd-8aa3-1841a4541b55"
 					(reference "FID3")
@@
 		)
 		(instances
-			(project "bitaxeSupra"
+			(project "bitaxeGamma"
 				(path "/e63e39d7-6ac0-4ffd-8aa3-1841a4541b55"
 					(reference "FID4")
@@
 		)
 		(instances
-			(project "bitaxeSupra"
+			(project "bitaxeGamma"
 				(path "/e63e39d7-6ac0-4ffd-8aa3-1841a4541b55"
 					(reference "FID6")
@@
 		)
 		(instances
-			(project "bitaxeSupra"
+			(project "bitaxeGamma"
 				(path "/e63e39d7-6ac0-4ffd-8aa3-1841a4541b55"
 					(reference "TP1")
@@
 		)
 		(instances
-			(project "bitaxeSupra"
+			(project "bitaxeGamma"
 				(path "/e63e39d7-6ac0-4ffd-8aa3-1841a4541b55"
 					(reference "TP2")
@@
 		)
 		(instances
-			(project "bitaxeSupra"
+			(project "bitaxeGamma"
 				(path "/e63e39d7-6ac0-4ffd-8aa3-1841a4541b55"
 					(reference "H8")
@@
 		)
 		(instances
-			(project "bitaxeSupra"
+			(project "bitaxeGamma"
 				(path "/e63e39d7-6ac0-4ffd-8aa3-1841a4541b55"
 					(reference "J1")
@@
 		)
 		(instances
-			(project "bitaxeSupra"
+			(project "bitaxeGamma"
 				(path "/e63e39d7-6ac0-4ffd-8aa3-1841a4541b55"
 					(reference "H1")
@@
 		)
 		(instances
-			(project "bitaxeSupra"
+			(project "bitaxeGamma"
 				(path "/e63e39d7-6ac0-4ffd-8aa3-1841a4541b55"
 					(reference "H7")
@@
 		)
 		(instances
-			(project "bitaxeSupra"
+			(project "bitaxeGamma"
 				(path "/e63e39d7-6ac0-4ffd-8aa3-1841a4541b55"
 					(reference "FID1")
@@
 		)
 		(instances
-			(project "bitaxeSupra"
+			(project "bitaxeGamma"
 				(path "/e63e39d7-6ac0-4ffd-8aa3-1841a4541b55"
 					(reference "FID8")
@@
 		)
 		(instances
-			(project "bitaxeSupra"
+			(project "bitaxeGamma"
 				(path "/e63e39d7-6ac0-4ffd-8aa3-1841a4541b55"
 					(reference "FID5")
@@
 		)
 		(instances
-			(project "bitaxeSupra"
+			(project "bitaxeGamma"
 				(path "/e63e39d7-6ac0-4ffd-8aa3-1841a4541b55"
 					(reference "H6")
@@
 		)
 		(instances
-			(project "bitaxeSupra"
+			(project "bitaxeGamma"
 				(path "/e63e39d7-6ac0-4ffd-8aa3-1841a4541b55"
 					(reference "FID7")
@@
 		)
 		(instances
-			(project "bitaxeSupra"
+			(project "bitaxeGamma"
 				(path "/e63e39d7-6ac0-4ffd-8aa3-1841a4541b55"
 					(reference "H5")
@@
 		)
 		(instances
-			(project "bitaxeSupra"
+			(project "bitaxeGamma"
 				(path "/e63e39d7-6ac0-4ffd-8aa3-1841a4541b55"
 					(reference "H3")
@@
 		)
 		(instances
-			(project "bitaxeSupra"
+			(project "bitaxeGamma"
 				(path "/e63e39d7-6ac0-4ffd-8aa3-1841a4541b55"
 					(reference "H2")
@@
 		)
 		(instances
-			(project "bitaxeSupra"
+			(project "bitaxeGamma"
 				(path "/e63e39d7-6ac0-4ffd-8aa3-1841a4541b55"
 					(reference "H4")
@@
 		)
 		(instances
-			(project "bitaxeSupra"
+			(project "bitaxeGamma"
 				(path "/e63e39d7-6ac0-4ffd-8aa3-1841a4541b55"
 					(reference "U1")
@@
 			(color 255 255 194 1.0000)
 		)
-		(property "Sheetname" "BM1368"
+		(property "Sheetname" "BM1370"
 			(at 113.03 71.6784 0)
 			(effects
@@
 			)
 		)
-		(property "Sheetfile" "bm1368.kicad_sch"
+		(property "Sheetfile" "bm1370.kicad_sch"
 			(at 113.03 91.0086 0)
 			(effects
@@
 		)
 		(instances
-			(project "bitaxeSupra"
+			(project "bitaxeGamma"
 				(path "/e63e39d7-6ac0-4ffd-8aa3-1841a4541b55"
 					(page "4")
@@
 		)
 		(instances
-			(project "bitaxeSupra"
+			(project "bitaxeGamma"
 				(path "/e63e39d7-6ac0-4ffd-8aa3-1841a4541b55"
 					(page "5")
@@
 		)
 		(instances
-			(project "bitaxeSupra"
+			(project "bitaxeGamma"
 				(path "/e63e39d7-6ac0-4ffd-8aa3-1841a4541b55"
 					(page "2")
@@
 		)
 		(instances
-			(project "bitaxeSupra"
+			(project "bitaxeGamma"
 				(path "/e63e39d7-6ac0-4ffd-8aa3-1841a4541b55"
 					(page "3")
