File: bitaxeGamma.kicad_sch (KiCad schematic)
At the start: 20 parts, among them J1 54-00164

Commit message: repair the heatsink mounting hole parts and nudge them back into a symmetrical pattern
Parts:
- H1, H2, H3, H4: footprint MountingHole:MountingHole_3mm_Pad_Via -> bitaxe:MountingHole_3mm_Pad_Via
- H5, H6: footprint MountingHole:MountingHole_3.5mm -> bitaxe:HeatsinkMountingHole_3mm
- H8: footprint MountingHole:MountingHole_3.5mm -> bitaxe:HeatsinkMountingHole_3.5mm
Changed lines of the file:
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@@
 			)
 		)
-		(property "Footprint" "MountingHole:MountingHole_3.5mm"
+		(property "Footprint" "bitaxe:HeatsinkMountingHole_3.5mm"
 			(at 66.04 189.23 0)
 			(effects
@@
 			)
 		)
-		(property "Footprint" "MountingHole:MountingHole_3mm_Pad_Via"
+		(property "Footprint" "bitaxe:MountingHole_3mm_Pad_Via"
 			(at 38.1 154.94 0)
 			(effects
@@
 			)
 		)
-		(property "Footprint" "MountingHole:MountingHole_3.5mm"
+		(property "Footprint" "bitaxe:HeatsinkMountingHole_3mm"
 			(at 66.04 174.625 0)
 			(effects
@@
 			)
 		)
-		(property "Footprint" "MountingHole:MountingHole_3.5mm"
+		(property "Footprint" "bitaxe:HeatsinkMountingHole_3mm"
 			(at 66.04 167.005 0)
 			(effects
@@
 			)
 		)
-		(property "Footprint" "MountingHole:MountingHole_3mm_Pad_Via"
+		(property "Footprint" "bitaxe:MountingHole_3mm_Pad_Via"
 			(at 38.1 171.45 0)
 			(effects
@@
 			)
 		)
-		(property "Footprint" "MountingHole:MountingHole_3mm_Pad_Via"
+		(property "Footprint" "bitaxe:MountingHole_3mm_Pad_Via"
 			(at 38.1 163.83 0)
 			(effects
@@
 			)
 		)
-		(property "Footprint" "MountingHole:MountingHole_3mm_Pad_Via"
+		(property "Footprint" "bitaxe:MountingHole_3mm_Pad_Via"
 			(at 38.1 179.07 0)
 			(effects
@@
 			(effects
 				(font
+					(size 1.27 1.27)
+				)
+				(hide yes)
+			)
+		)
+		(property "exclude_from_bom" ""
+			(at 0 318.77 0)
+			(effects
+				(font
