File: bm1370.kicad_sch (KiCad schematic)
At the start: 49 parts, among them U5 MCP1824T-1202E/OT, U6 MCP1824T-0802E, U7 25MHz, U8 BM1368_mode1, U9 SN74AVC4T774

Commit message: switching to gamma/600 naming
Parts:
- U8: value BM1368_mode1 -> BM1370_mode1; footprint bitaxe:BM1368 -> (none); symbol bitaxe:BM1368_mode1 -> bitaxe:BM1370_mode1
Other:
- title: bitaxeSupra -> bitaxeGamma
