File: bm1370.kicad_sch (KiCad schematic)
At the start: 49 parts, among them U5 MCP1824T-1202E/OT, U6 MCP1824T-0802E, U7 25MHz, U8 BM1370_mode1, U9 SN74AVC4T774

Commit message: added BM1370 footprint
Parts:
- U8: footprint (none) -> bitaxe:BM1370
Changed lines of the file:
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@@
 			)
 		)
-		(property "Footprint" ""
+		(property "Footprint" "bitaxe:BM1370"
 			(at 157.48 144.78 0)
 			(effects

Commit message: BOM update
Parts:
- C43: DK 1276-1782-2-ND -> 1276-1782-1-ND
Changed lines of the file:
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@@
 			)
 		)
-		(property "DK" "1276-1782-2-ND"
+		(property "DK" "1276-1782-1-ND"
 			(at 147.32 57.15 0)
 			(effects

Commit message: fix oscillator name
Parts:
- U7: footprint bitaxe:O 25,0-JO32-B-1V3-1-T1-LF -> bitaxe:SMD3225-4P
Changed lines of the file:
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@@
 			)
 		)
-		(property "Footprint" "bitaxe:O 25,0-JO32-B-1V3-1-T1-LF"
+		(property "Footprint" "bitaxe:SMD3225-4P"
 			(at 40.64 172.72 0)
 			(effects
