File: esp32.kicad_sch (KiCad schematic)
At the start: 21 parts, among them J2 TC2030-IDC, J3 Conn_01x04, J4 Conn_01x06, J5 USB_C_Receptacle_USB2.0, SW1 GT-TC029B-H025-L1N, SW2 GT-TC029B-H025-L1N, U3 RT9080-33GJ5, U4 ESP32-S3-WROOM-1

Commit message: remove J3 from BOM for #2
Parts:
- J3: DK S5596-ND -> (none); PARTNO NPTC041KFXC-RC -> (none); now left out of the parts list
Changed lines of the file:
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@@
 		(unit 1)
 		(exclude_from_sim no)
-		(in_bom yes)
+		(in_bom no)
 		(on_board yes)
 		(dnp no)
@@
 			(at 196.85 32.385 0)
 			(effects
-				(font
-					(size 1.27 1.27)
-				)
-				(hide yes)
-			)
-		)
-		(property "DK" "S5596-ND"
-			(at 196.85 32.385 0)
-			(effects
-				(font
-					(size 1.27 1.27)
-				)
-				(hide yes)
-			)
-		)
-		(property "PARTNO" "NPTC041KFXC-RC"
-			(at 196.85 32.385 0)
-			(effects

Commit message: repair the heatsink mounting hole parts and nudge them back into a symmetrical pattern
Parts:
- J3: DK (none) -> S5596-ND; PARTNO (none) -> NPTC041KFXC-RC
Changed lines of the file:
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@@
+			)
+		)
+		(property "DK" "S5596-ND"
+			(at 0 64.77 0)
+			(effects
+				(font
+					(size 1.27 1.27)
+				)
+				(hide yes)
+			)
+		)
+		(property "PARTNO" "NPTC041KFXC-RC"
+			(at 0 64.77 0)
+			(effects
+				(font
+					(size 1.27 1.27)
+				)
+				(hide yes)
 			)
 		)
@@
 			(effects
 				(font
+					(size 1.27 1.27)
+				)
+				(hide yes)
+			)
+		)
+		(property "exclude_from_bom" ""
+			(at 0 337.82 0)
+			(effects
+				(font
