File: fan.kicad_sch (KiCad schematic)
At the start: 14 parts, among them J6 Conn_01x04, U10 EMC2101

Commit message: switching to gamma/600 naming
Other:
- title: bitaxeSupra -> bitaxeGamma
Changed lines of the file:
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@@
 	(paper "A")
 	(title_block
-		(title "bitaxeSupra")
-		(date "2024-04-07")
-		(rev "402")
+		(title "bitaxeGamma")
+		(date "2024-07-02")
+		(rev "600x")
 	)
 	(junction
@@
 		)
 		(instances
-			(project "bitaxeSupra"
+			(project "bitaxeGamma"
 				(path "/e63e39d7-6ac0-4ffd-8aa3-1841a4541b55/8e8832ea-6bf1-49d2-b3a5-32a207f555d2"
 					(reference "TP38")
@@
 				)
 			)
-			(project "bitaxeSupra"
+			(project "bitaxeGamma"
 				(path "/e63e39d7-6ac0-4ffd-8aa3-1841a4541b55/8e8832ea-6bf1-49d2-b3a5-32a207f555d2"
 					(reference "R24")
@@
 		)
 		(instances
-			(project "bitaxeSupra"
+			(project "bitaxeGamma"
 				(path "/e63e39d7-6ac0-4ffd-8aa3-1841a4541b55/8e8832ea-6bf1-49d2-b3a5-32a207f555d2"
 					(reference "C53")
@@
 		)
 		(instances
-			(project "bitaxeSupra"
+			(project "bitaxeGamma"
 				(path "/e63e39d7-6ac0-4ffd-8aa3-1841a4541b55/8e8832ea-6bf1-49d2-b3a5-32a207f555d2"
 					(reference "C52")
@@
 		)
 		(instances
-			(project "bitaxeSupra"
+			(project "bitaxeGamma"
 				(path "/e63e39d7-6ac0-4ffd-8aa3-1841a4541b55/8e8832ea-6bf1-49d2-b3a5-32a207f555d2"
 					(reference "R22")
@@
 		)
 		(instances
-			(project "bitaxeSupra"
+			(project "bitaxeGamma"
 				(path "/e63e39d7-6ac0-4ffd-8aa3-1841a4541b55/8e8832ea-6bf1-49d2-b3a5-32a207f555d2"
 					(reference "C50")
@@
 		)
 		(instances
-			(project "bitaxeSupra"
+			(project "bitaxeGamma"
 				(path "/e63e39d7-6ac0-4ffd-8aa3-1841a4541b55/8e8832ea-6bf1-49d2-b3a5-32a207f555d2"
 					(reference "C51")
@@
 		)
 		(instances
-			(project "bitaxeSupra"
+			(project "bitaxeGamma"
 				(path "/e63e39d7-6ac0-4ffd-8aa3-1841a4541b55/8e8832ea-6bf1-49d2-b3a5-32a207f555d2"
 					(reference "TP35")
@@
 		)
 		(instances
-			(project "bitaxeSupra"
+			(project "bitaxeGamma"
 				(path "/e63e39d7-6ac0-4ffd-8aa3-1841a4541b55/8e8832ea-6bf1-49d2-b3a5-32a207f555d2"
 					(reference "J6")
@@
 		)
 		(instances
-			(project "bitaxeSupra"
+			(project "bitaxeGamma"
 				(path "/e63e39d7-6ac0-4ffd-8aa3-1841a4541b55/8e8832ea-6bf1-49d2-b3a5-32a207f555d2"
 					(reference "TP36")
@@
 		)
 		(instances
-			(project "bitaxeSupra"
+			(project "bitaxeGamma"
 				(path "/e63e39d7-6ac0-4ffd-8aa3-1841a4541b55/8e8832ea-6bf1-49d2-b3a5-32a207f555d2"
 					(reference "R23")
@@
 		)
 		(instances
-			(project "bitaxeSupra"
+			(project "bitaxeGamma"
 				(path "/e63e39d7-6ac0-4ffd-8aa3-1841a4541b55/8e8832ea-6bf1-49d2-b3a5-32a207f555d2"
 					(reference "TP37")
@@
 		)
 		(instances
-			(project "bitaxeSupra"
+			(project "bitaxeGamma"
 				(path "/e63e39d7-6ac0-4ffd-8aa3-1841a4541b55/8e8832ea-6bf1-49d2-b3a5-32a207f555d2"
 					(reference "R25")
@@
 		)
 		(instances
-			(project "bitaxeSupra"
+			(project "bitaxeGamma"
 				(path "/e63e39d7-6ac0-4ffd-8aa3-1841a4541b55/8e8832ea-6bf1-49d2-b3a5-32a207f555d2"
 					(reference "U10")
