File: power.kicad_sch (KiCad schematic)
At the start: 40 parts, among them T1 net-tie, U2 TPS546D24ARVFR

Commit message: BOM update
Parts:
- C17, C18, C19, C20: DK 1276-1782-2-ND -> 1276-1782-1-ND
Changed lines of the file:
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@@
 			)
 		)
-		(property "DK" "1276-1782-2-ND"
+		(property "DK" "1276-1782-1-ND"
 			(at 224.79 68.58 0)
 			(effects
@@
 			)
 		)
-		(property "DK" "1276-1782-2-ND"
+		(property "DK" "1276-1782-1-ND"
 			(at 214.63 60.96 0)
 			(effects
@@
 			)
 		)
-		(property "DK" "1276-1782-2-ND"
+		(property "DK" "1276-1782-1-ND"
 			(at 234.95 60.96 0)
 			(effects
@@
 			)
 		)
-		(property "DK" "1276-1782-2-ND"
+		(property "DK" "1276-1782-1-ND"
 			(at 204.47 68.58 0)
 			(effects

Commit message: repair the heatsink mounting hole parts and nudge them back into a symmetrical pattern
Parts:
- T1: DK (none) -> P16200CT-ND; PARTNO (none) -> 2R5TPE220MAFB
Changed lines of the file:
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@@
+			)
+		)
+		(property "DK" "P16200CT-ND"
+			(at 0 281.94 0)
+			(effects
+				(font
+					(size 1.27 1.27)
+				)
+				(hide yes)
+			)
+		)
+		(property "PARTNO" "2R5TPE220MAFB"
+			(at 0 281.94 0)
+			(effects
+				(font
+					(size 1.27 1.27)
+				)
+				(hide yes)
 			)
 		)
